Commit message: temporary dummy interia value to pass gz fortress parsing

File: tiago_description/urdf/arm/arm.urdf.xacro (robot description, xacro)
@@ -41,7 +41,12 @@
       <inertial>
         <!--<origin xyz="0.061191 ${reflect * -0.022397} -0.012835" rpy="0.00000 0.00000 0.00000"/>-->
-        <origin xyz="0.061191 -0.022397 ${reflect * -0.012835}" rpy="0.00000 0.00000 0.00000"/>
-        <mass value="1.563428"/>
-        <inertia ixx="0.002471" ixy="${reflect * -0.001809}" ixz="-0.001202" iyy="0.006132" iyz="${reflect * 0.000494}" izz="0.006704"/>
+        <!--<origin xyz="0.061191 -0.022397 ${reflect * -0.012835}" rpy="0.00000 0.00000 0.00000"/>-->
+        <!-- <origin xyz="0.061191 -0.022397 0.012835" rpy="0.00000 0.00000 0.00000"/> -->
+        <!-- <mass value="1.563428"/> -->
+        <!--<inertia ixx="0.002471" ixy="${reflect * -0.001809}" ixz="-0.001202" iyy="0.006132" iyz="${reflect * 0.000494}" izz="0.006704"/>-->
+        <!-- <inertia ixx="0.002471" ixy="0.001809" ixz="-0.001202" iyy="0.006132" iyz="-0.000494" izz="0.006704"/>-->
+        <origin xyz="0.0 0.0 0.0" rpy="0.0 0.0 0.0"/>
+        <mass value="1.0"/>
+        <inertia ixx="0.01" ixy="0.0" ixz="0.0" iyy="0.01" iyz="0.0" izz="0.01"/>
       </inertial>
       <!-- M90 module -->

Commit message: meshlab inertia values

File: tiago_description/urdf/arm/arm.urdf.xacro (robot description, xacro)
@@ -40,13 +40,10 @@
     <link name="${name}_1_link">
       <inertial>
+      <!-- Intertia patch -->
         <!--<origin xyz="0.061191 ${reflect * -0.022397} -0.012835" rpy="0.00000 0.00000 0.00000"/>-->
-        <!--<origin xyz="0.061191 -0.022397 ${reflect * -0.012835}" rpy="0.00000 0.00000 0.00000"/>-->
-        <!-- <origin xyz="0.061191 -0.022397 0.012835" rpy="0.00000 0.00000 0.00000"/> -->
-        <!-- <mass value="1.563428"/> -->
+        <origin xyz="0.061191 -0.022397 ${reflect * -0.012835}" rpy="0.00000 0.00000 0.00000"/>
+        <mass value="1.563428"/>
         <!--<inertia ixx="0.002471" ixy="${reflect * -0.001809}" ixz="-0.001202" iyy="0.006132" iyz="${reflect * 0.000494}" izz="0.006704"/>-->
-        <!-- <inertia ixx="0.002471" ixy="0.001809" ixz="-0.001202" iyy="0.006132" iyz="-0.000494" izz="0.006704"/>-->
-        <origin xyz="0.0 0.0 0.0" rpy="0.0 0.0 0.0"/>
-        <mass value="1.0"/>
-        <inertia ixx="0.01" ixy="0.0" ixz="0.0" iyy="0.01" iyz="0.0" izz="0.01"/>
+        <inertia ixx="0.0030552108" ixy="${reflect * -0.0019074323}" ixz="0.0015792527" iyy="0.0066930687" iyz="${reflect * 0.0006810805}" izz="0.0070890817"/>
       </inertial>
       <!-- M90 module -->
